Commit message: Attempt ROS2 Robot Support Package

File: atturtle_description/urdf/common_properties.xacro (robot description, xacro)
@@ -15,3 +15,8 @@
         </material>
     </xacro:property>
+    <xacro:property name="material_green">
+        <material name="green">
+            <color rgba="0.0 0.8 0 1" />
+        </material>
+    </xacro:property>
 </robot>
