Commit message: Convert to ROS1 - Noetic

File: atturtle_description/urdf/atturtle.xacro (robot description, xacro)
@@ -1,5 +1,5 @@
-?xml version="1.0" ?>
+<?xml version="1.0" ?>
 <robot name="atturtle" xmlns:xacro="http://ros.org/wiki/xacro">
-  <xacro:include filename="$(find atturtle_description)/urdf/atturtle_macro.xacro" />
-  <xacro:atturtle prefix=""/>
+    <xacro:include filename="$(find atturtle_description)/urdf/atturtle_macro.xacro" />
+    <xacro:atturtle prefix=""/>
 </robot>

File: atturtle_description/urdf/atturtle_macro.xacro (robot description, xacro)
@@ -1,6 +1,6 @@
 <?xml version="1.0" ?>
 <robot xmlns:xacro="http://ros.org/wiki/xacro">
-<xacro:macro name="motoman_ms210" params="prefix">
-    <xacro:include filename="$(find motoman_resources)/urdf/common_materials.xacro"/>
+<xacro:macro name="atturtle" params="prefix">
+    <xacro:include filename="$(find atturtle_description)/urdf/common_properties.xacro"/>
     <!-- link list -->
     <!-- base_footprint is a fictitious link(frame) that is on the ground right below link_base origin, navigation stack depends on this frame -->
@@ -22,14 +22,14 @@
     <link  name="${prefix}link_base">
         <visual>
-            <origin xyz="0 0 0.0.0127" rpy="0 0 0" />
+            <origin xyz="0 0 0.025" rpy="0 0 0" />
             <geometry>
-                <cylinder length="0.2" radius="0.15875"/>
+                <cylinder length="0.0635" radius="0.15875"/>
             </geometry>
             <xacro:material_light_grey/>
         </visual>
         <collision>
-            <origin xyz="0 0 0" rpy="0 0 0" />
+            <origin xyz="0 0 0.025" rpy="0 0 0" />
             <geometry>
-                <cylinder length="0.2" radius="0.15875"/>
+                <cylinder length="0.0635" radius="0.15875"/>
             </geometry>
         </collision>
@@ -85,5 +85,5 @@
     </joint>
     <joint name="${prefix}left_wheel_joint" type="continuous">
-	    <origin xyz="0 0.13 0.015" rpy="0 0 0"/>
+	    <origin xyz="0 0.1016 0.015" rpy="0 0 0"/>
 	    <parent link="${prefix}link_base"/>
 	    <child link="${prefix}left_wheel_link"/>
@@ -91,5 +91,5 @@
     </joint>
     <joint name="${prefix}right_wheel_joint" type="continuous">
-	    <origin xyz="0 -0.13 0.015" rpy="0 0 0"/>
+	    <origin xyz="0 -0.1016 0.015" rpy="0 0 0"/>
 	    <parent link="${prefix}link_base"/>
 	    <child link="${prefix}right_wheel_link"/>
@@ -97,6 +97,6 @@
     </joint>
     <joint name="${prefix}rear_castor_joint" type="fixed">
-	    <origin xyz="-0.13 0 0.0" rpy="0 0 0"/>
-	    <parent link="${prefix}base_link"/>
+	    <origin xyz="0.1143 0 0" rpy="0 0 0"/>
+	    <parent link="${prefix}link_base"/>
 	    <child link="${prefix}rear_wheel_link"/>
 	    <axis xyz="0 1 0"/>

File: atturtle_description/urdf/common_properties.xacro (robot description, xacro)
@@ -3,20 +3,19 @@
   Various useful properties such as constants and materials
  -->
-<robot name="xacro_properties" xmlns:xacro="http://ros.org/wiki/xacro">
-    <xacro:property name="M_PI" value="3.1415926535897931" />
-    <xacro:property name="material_light_grey">
+<robot xmlns:xacro="http://ros.org/wiki/xacro">
+    <xacro:macro name="material_light_grey">
         <material name="light_grey">
             <color rgba="0.6 0.6 0.6 1" />
         </material>
-    </xacro:property>
-    <xacro:property name="material_black">
+    </xacro:macro>
+    <xacro:macro name="material_black">
         <material name="black">
             <color rgba="0.1 0.1 0.1 1" />
         </material>
-    </xacro:property>
-    <xacro:property name="material_green">
+    </xacro:macro>
+    <xacro:macro name="material_green">
         <material name="green">
             <color rgba="0.0 0.8 0 1" />
         </material>
-    </xacro:property>
+    </xacro:macro>
 </robot>
