Commit message: Add Joint Effort & Velocity Limits

File: atturtle_description/urdf/atturtle_macro.xacro (robot description, xacro)
@@ -89,4 +89,6 @@
 	    <child link="${prefix}left_wheel_link"/>
 	    <axis xyz="0 1 0"/>
+        <limit effort="100" velocity="100"/>
+        <joint_properties damping="0.0" friction="0.0"/>
     </joint>
     <joint name="${prefix}right_wheel_joint" type="continuous">
@@ -95,4 +97,6 @@
 	    <child link="${prefix}right_wheel_link"/>
 	    <axis xyz="0 1 0"/>
+        <limit effort="100" velocity="100"/>
+        <joint_properties damping="0.0" friction="0.0"/>
     </joint>
     <joint name="${prefix}rear_castor_joint" type="fixed">
